File: kicad/_autosave-Bluetooth_RN4020.kicad_pcb (KiCad board)
At the start: 2 copper layers, 9 parts, among them U1 RN4020

Commit message: Casi listo
Parts:
- added G***: LOGO, Poncho_Esqueleto:Logo_Poncho, F.Cu at (148.8, 70.8)
- added G***: Logo_EDU-CIAA, Poncho_Esqueleto:Logo_EDU-CIAA, F.Cu at (162.3, 71.1)
- moved D1 4.00 mm to (136.8, 97.5)
- moved R1 4.00 mm to (145.8, 97.5)
- moved D2 2.00 mm to (136.8, 104.5)
- moved R2 2.00 mm to (145.8, 104.5)
Routing:
- net (no net): track 0.00 -> 335.7 mm
- net CMD: track 80.2 -> 90.4 mm
- net SW: track 89.5 -> 99.3 mm
- net Net-(R1-Pad1): track 28.1 -> 32.1 mm
- net Net-(R2-Pad1): track 21.1 -> 23.1 mm
Other:
- board text added: "+3.3V"
- board text added: "Awake"
- board text added: "Connected"
- board text added: "Event"
- board text added: "Laurella Morgillo Muriel Solito Zubieta"
