File: kicad/Bluetooth_RN4020.kicad_pcb (KiCad board)
At the start: 2 copper layers, 0 parts

Commit message: Limpieza
Parts:
- added C1: C, SM1206POL, F.Cu at (144.8, 87.6)
- added D1: LED, LED-3MM, F.Cu at (118.1, 127.0)
- added D2: LED, LED-3MM, F.Cu at (129.5, 125.7)
- added D3: LED, LED-3MM, F.Cu at (142.2, 125.7)
- added R1: R, SM1206, F.Cu at (115.6, 113.0)
- added R2: R, SM1206, F.Cu at (124.5, 109.2)
- added R3: R, SM1206, F.Cu at (138.4, 111.8)
- added U1: RN4020, RN4020, F.Cu at (124.5, 95.2)

Commit message: FUSION
Parts:
- added G***: Logo_EDU-CIAA, Poncho_Esqueleto:Logo_EDU-CIAA, F.Cu at (427.0, 74.2)
- added G***: LOGO, Poncho_Esqueleto:Logo_Poncho, F.Cu at (403.5, 74.2)
- added G101: Logo_OSHWA, Poncho_Esqueleto:Logo_OSHWA, F.Cu at (414.3, 74.2)
- added MP?: Plantilla_EDU-CIAA, Poncho_Esqueleto:Plantilla_EDU-CIAA, F.Cu at (454.9, 54.5)
- added P1: CONN_5, Poncho_Modelos:bornier5, F.Cu at (420.6, 51.9)
- added P2: CONN_4, Poncho_Modelos:bornier4, F.Cu at (420.6, 95.1)
- added XA1: Conn_PonchoMP_2x_20x2, Poncho_Esqueleto:Conn_Poncho_Chico, F.Cu at (454.9, 54.5)
- moved R1 12.0 mm to (121.9, 102.9)
- moved D3 11.5 mm to (134.7, 117.0)
- moved D1 10.7 mm to (122.0, 117.0)
- moved R3 9.73 mm to (134.5, 102.8)
- moved D2 8.78 mm to (128.4, 117.0)
- moved R2 7.41 mm to (128.3, 102.9)
- moved C1 4.12 mm to (146.1, 83.7), turned to 90 degrees
Routing:
- net GND: track 0.00 -> 155.8 mm
- net +5VP: track 0.00 -> 73.3 mm
- net Net-(P1-Pad4): track 0.00 -> 60.1 mm
- net Net-(P1-Pad3): track 0.00 -> 54.7 mm
- net +3.3V: track 0.00 -> 45.2 mm
- net Net-(P2-Pad3): track 0.00 -> 43.4 mm
- net Net-(P2-Pad2): track 0.00 -> 36.9 mm
- net +5V: track 0.00 -> 28.8 mm
- net N-0000018: track 0.00 -> 13.7 mm
- net N-0000017: track 0.00 -> 13.6 mm
- net N-0000016: track 0.00 -> 13.6 mm
- net N-0000020: track 0.00 -> 10.8 mm
- net N-0000019: track 0.00 -> 10.3 mm
- net N-000007: track 0.00 -> 6.47 mm
Other:
- board outline added: 86.4 x 61 mm
- net class Default: clearance 0.254 -> 0.508; trace_width 0.254 -> 0.381; via_dia 0.889 -> 0.6; via_drill 0.635 -> 0.4
- rule pad_to_mask_clearance: 0 -> 0.2
- rule trace_clearance: 0.254 -> 0.508
- rule trace_min: 0.254 -> 0.2
- rule via_min_drill: 0.508 -> 0.3
- rule via_min_size: 0.889 -> 0.4
- board text added: "Borrar (Footprint MP1) la Plantilla-EDU-CIAA al finalizar el posicionamiento y definido el borde de PCB."
- board text added: "Diseño simple faz. Sin requerimientos especiales."
- board text added: "Editar el rótulo"
- board text added: "Editar el stackup para reflejar cantidad de capas, si se han realizado cálculos de impedancia o si es relevante para el funcionamiento."
- board text added: "PONCHO CHICO"
- board text added: "PONCHO CHICO http://www.proyecto-ciaa.com.ar/"
- board text added: "Para un diseño nuevo luego de modificar el esquemático: 1)Seleccionar el bloque del PCB y cotas. (click-drag-release). 2)Opción de borrar bloque (Botón derecho). 3)Marcar todo menos locked footprints (MP1 y XA1) 4) Aceptar. 5) Volver a cargar el netlist."
- board text added: "STACK-UP"
- board text added: "Se sugiere colocar código de Poncho en cobre, serigrafía y rótulo."
- board text added: "www.proyecto-ciaa.com.ar"

Commit message: Poncho Mediano
Parts:
- removed G***: Logo_EDU-CIAA, Poncho_Esqueleto:Logo_EDU-CIAA
- removed G***: LOGO, Poncho_Esqueleto:Logo_Poncho
- removed G101: Logo_OSHWA, Poncho_Esqueleto:Logo_OSHWA
- removed MP?: Plantilla_EDU-CIAA, Poncho_Esqueleto:Plantilla_EDU-CIAA
- removed P1: CONN_5, Poncho_Modelos:bornier5
- removed P2: CONN_4, Poncho_Modelos:bornier4
- XA1: footprint Poncho_Esqueleto:Conn_Poncho_Chico -> Poncho_Esqueleto:Conn_Poncho_Mediano
- moved XA1 269.9 mm to (185.2, 64.0)
- moved D1 51.8 mm to (169.4, 96.1), turned to 270 degrees
- moved R1 48.1 mm to (169.5, 110.2), turned to 90 degrees
- moved C1 47.8 mm to (140.5, 131.2)
- moved U1 42.2 mm to (156.1, 123.2), turned to 180 degrees
- moved D2 40.5 mm to (163.0, 96.1), turned to 270 degrees
- moved R2 35.6 mm to (163.1, 110.2), turned to 90 degrees
- moved D3 30.4 mm to (156.7, 96.1), turned to 270 degrees
- moved R3 23.6 mm to (156.9, 110.2), turned to 90 degrees
Connections:
- U1 pad 13: (no net) -> N-000004
- U1 pad 14: (no net) -> CTS
- U1 pad 15: (no net) -> HW
- U1 pad 17: (no net) -> N-000005
- U1 pad 18: (no net) -> RTS
- U1 pad 19: (no net) -> N-000006
- U1 pad 2: (no net) -> N-000001
- U1 pad 20: (no net) -> N-0000024
- U1 pad 21: (no net) -> N-0000023
- U1 pad 22: (no net) -> N-0000022
- U1 pad 3: (no net) -> N-000002
- U1 pad 4: (no net) -> N-000003
- U1 pad 5: (no net) -> UART_TX
- U1 pad 6: (no net) -> UART_RX
- U1 pad 7: (no net) -> SW
- U1 pad 8: (no net) -> CMD
- XA1 pad 44: (no net) -> Net-(P2-Pad3)
- XA1 pad 56: (no net) -> Net-(P2-Pad2)
- XA1 pad 72: Net-(P2-Pad3) -> (no net)
- XA1 pad 74: Net-(P2-Pad2) -> (no net)
Routing:
- net GND: track 155.8 -> 20.9 mm
- net +5VP: track 73.3 -> 0.00 mm
- net Net-(P1-Pad4): track 60.1 -> 0.00 mm
- net Net-(P1-Pad3): track 54.7 -> 0.00 mm
- net Net-(P2-Pad3): track 43.4 -> 0.00 mm
- net +3.3V: track 45.2 -> 4.34 mm
- net Net-(P2-Pad2): track 36.9 -> 0.00 mm
- net +5V: track 28.8 -> 0.00 mm
Other:
- board outline removed
- net class Default: clearance 0.508 -> 0.25
- rule trace_clearance: 0.508 -> 0.25
- board text removed: "Borrar (Footprint MP1) la Plantilla-EDU-CIAA al finalizar el posicionamiento y definido el borde de PCB."
- board text removed: "Diseño simple faz. Sin requerimientos especiales."
- board text removed: "Editar el rótulo"
- board text removed: "Editar el stackup para reflejar cantidad de capas, si se han realizado cálculos de impedancia o si es relevante para el funcionamiento."
- board text removed: "PONCHO CHICO"
- board text removed: "PONCHO CHICO http://www.proyecto-ciaa.com.ar/"
- board text removed: "Para un diseño nuevo luego de modificar el esquemático: 1)Seleccionar el bloque del PCB y cotas. (click-drag-release). 2)Opción de borrar bloque (Botón derecho). 3)Marcar todo menos locked footprints (MP1 y XA1) 4) Aceptar. 5) Volver a cargar el netlist."
- board text removed: "STACK-UP"
- board text removed: "Se sugiere colocar código de Poncho en cobre, serigrafía y rótulo."
- board text removed: "www.proyecto-ciaa.com.ar"

Commit message: 50% Poncho
Parts:
- C1: footprint SM1206POL -> Capacitors_Tantalum_SMD:TantalC_SizeB_EIA-3528_Reflow
- R1, R2, R3: footprint SM1206 -> Resistors_SMD:R_1206
- moved D1 18.3 mm to (165.4, 113.9), turned to 180 degrees
- moved R1 13.6 mm to (156.4, 113.9), turned to 0 degrees
- moved D2 13.0 mm to (165.4, 108.9), turned to 180 degrees
- moved D3 11.7 mm to (165.4, 103.9), turned to 180 degrees
- moved R2 6.92 mm to (156.4, 108.9), turned to 0 degrees
- moved R3 6.37 mm to (156.4, 103.9), turned to 0 degrees
- moved C1 4.38 mm to (136.2, 130.4), turned to 270 degrees
- moved XA1 0.97 mm to (185.2, 65.0)
- moved U1 0.81 mm to (156.0, 124.0)
Routing:
- net GND: track 20.9 -> 38.5 mm, vias 0 -> 2
- net N-0000019: track 10.3 -> 25.6 mm
- net N-000007: track 6.47 -> 17.7 mm
- net +3.3V: track 4.34 -> 11.8 mm
- net N-0000018: track 13.7 -> 6.28 mm
- net N-0000017: track 13.6 -> 6.28 mm
- net N-0000016: track 13.6 -> 6.28 mm

Commit message: New Poncho
Parts:
- C1: value C -> CP1
Connections:
- C1 pad 1: +3.3V -> +3V3
- U1 pad 23: +3.3V -> +3V3
- U1 pad 5: UART_TX -> TX
- U1 pad 6: UART_RX -> RX
- XA1 pad 1: +3.3V -> (no net)
- XA1 pad 2: +5V -> (no net)
- XA1 pad 23: Net-(P1-Pad3) -> RX
- XA1 pad 25: Net-(P1-Pad4) -> TX
- XA1 pad 42: +5VP -> (no net)
- XA1 pad 43: GND -> (no net)
- XA1 pad 44: Net-(P2-Pad3) -> (no net)
- XA1 pad 45: GND -> (no net)
- XA1 pad 47: GND -> (no net)
- XA1 pad 56: Net-(P2-Pad2) -> (no net)
- XA1 pad 69: (no net) -> Net-(XA1-Pad69)
- XA1 pad 71: (no net) -> Net-(XA1-Pad71)
- XA1 pad 72: (no net) -> SW
- XA1 pad 73: (no net) -> Net-(XA1-Pad73)
- XA1 pad 74: (no net) -> CMD
- XA1 pad 75: (no net) -> Net-(XA1-Pad75)
- XA1 pad 76: (no net) -> CTS
- XA1 pad 77: GND -> (no net)
- XA1 pad 78: (no net) -> HW
- XA1 pad 79: GND -> (no net)
- XA1 pad 80: (no net) -> RTS
Routing:
- net RTS: track 0.00 -> 36.9 mm
- net GND: track 38.5 -> 23.1 mm, vias 2 -> 4
- net +3V3: track 0.00 -> 11.8 mm
- net +3.3V: track 11.8 -> 0.00 mm
- added copper zone on B.Cu, net GND
Other:
- net class Default: clearance 0.25 -> 0.1
- rule trace_clearance: 0.25 -> 0.1

Commit message: PCB Completa
Parts:
- moved D1 31.2 mm to (136.8, 101.5), turned to 0 degrees
- moved D3 29.6 mm to (136.8, 111.5), turned to 0 degrees
- moved D2 28.7 mm to (136.8, 106.5), turned to 0 degrees
- moved R1 16.4 mm to (145.8, 101.5), turned to 180 degrees
- moved R3 13.0 mm to (145.8, 111.5), turned to 180 degrees
- moved R2 10.9 mm to (145.8, 106.5), turned to 180 degrees
- moved C1 0.79 mm to (136.2, 131.2), turned to 180 degrees
Connections:
- XA1 pad 41: (no net) -> +3V3
- XA1 pad 42: (no net) -> Net-(XA1-Pad42)
- XA1 pad 43: (no net) -> Net-(XA1-Pad43)
- XA1 pad 45: (no net) -> Net-(XA1-Pad45)
- XA1 pad 47: (no net) -> Net-(XA1-Pad47)
- XA1 pad 51: (no net) -> Net-(XA1-Pad51)
- XA1 pad 53: (no net) -> Net-(XA1-Pad53)
- XA1 pad 57: (no net) -> Net-(XA1-Pad57)
- XA1 pad 59: (no net) -> Net-(XA1-Pad59)
- XA1 pad 65: (no net) -> Net-(XA1-Pad65)
- XA1 pad 67: (no net) -> Net-(XA1-Pad67)
- XA1 pad 77: (no net) -> Net-(XA1-Pad77)
- XA1 pad 79: (no net) -> GND
Routing:
- net +3V3: track 11.8 -> 106.0 mm
- net SW: track 0.00 -> 89.5 mm
- net CMD: track 0.00 -> 80.2 mm
- net RX: track 0.00 -> 60.0 mm
- net TX: track 0.00 -> 59.6 mm
- net CTS: track 0.00 -> 40.7 mm
- net HW: track 0.00 -> 37.7 mm
- net Net-(R1-Pad1): track 10.5 -> 28.1 mm
- net Net-(R3-Pad1): track 25.6 -> 13.8 mm
- net Net-(R2-Pad1): track 17.7 -> 21.1 mm
- net GND: track 23.1 -> 26.0 mm, vias 4 -> 6
- net RTS: track 36.9 -> 38.9 mm

Commit message: Casi listo
Parts:
- moved D1 4.00 mm to (136.8, 97.5)
- moved R1 4.00 mm to (145.8, 97.5)
- moved D2 2.00 mm to (136.8, 104.5)
- moved R2 2.00 mm to (145.8, 104.5)
Routing:
- net (no net): track 0.00 -> 335.7 mm
- net CMD: track 80.2 -> 90.4 mm
- net SW: track 89.5 -> 99.3 mm
- net Net-(R1-Pad1): track 28.1 -> 32.1 mm
- net Net-(R2-Pad1): track 21.1 -> 23.1 mm
Other:
- board text added: "+3.3V"
- board text added: "Awake"
- board text added: "Connected"
- board text added: "Event"
- board text added: "Laurella Morgillo Muriel Solito Zubieta"

Commit message: Ploteo
Parts:
- added G***: Logo_EDU-CIAA, Poncho_Esqueleto:Logo_EDU-CIAA, F.Cu at (155.5, 71.2)
Routing:
- net SW: track 99.3 -> 96.5 mm
- net CMD: track 90.4 -> 87.8 mm
- net RX: track 60.0 -> 57.9 mm
- net TX: track 59.6 -> 57.9 mm
Other:
- board text removed: "Laurella Morgillo Muriel Solito Zubieta"
