File: kicad/Bluetooth_RN4020.sch (KiCad schematic (older format))
At the start: 8 parts, among them U1 RN4020

Commit message: FUSION
Connections:
- wire segments 30 -> 32
Changed lines of the file:
@@
 LIBS:memory
 LIBS:xilinx
-LIBS:special
 LIBS:microcontrollers
 LIBS:dsp
@@
 LIBS:RN4020
 LIBS:Bluetooth_RN4020-cache
-EELAYER 27 0
+EELAYER 25 0
 EELAYER END
 $Descr A4 11693 8268
@@
 Text GLabel 3950 6050 3    60   Input ~ 0
 HW
-$Comp
-L RN4020 U1
-U 1 1 561FC38B
-P 3450 4400
-F 0 "U1" H 2800 5350 60  0001 C CNN
-F 1 "RN4020" H 3950 5350 60  0000 C CNN
-F 2 "" H 3950 5350 60  0001 C CNN
-F 3 "" H 3950 5350 60  0000 C CNN
-	1    3450 4400
-	1    0    0    -1
-$EndComp
 Wire Wire Line
 	3500 7250 3500 7100
@@
 L GND #PWR03
 U 1 1 561FD06E
-P 4000 5550
-F 0 "#PWR03" H 4000 5300 50  0001 C CNN
-F 1 "GND" H 4000 5400 50  0000 C CNN
-F 2 "" H 4000 5550 60  0000 C CNN
-F 3 "" H 4000 5550 60  0000 C CNN
-	1    4000 5550
+P 4000 5600
+F 0 "#PWR03" H 4000 5350 50  0001 C CNN
+F 1 "GND" H 4000 5450 50  0000 C CNN
+F 2 "" H 4000 5600 60  0000 C CNN
+F 3 "" H 4000 5600 60  0000 C CNN
+	1    4000 5600
 	1    0    0    -1
 $EndComp
@@
 L GND #PWR04
 U 1 1 561FD154
-P 2850 5550
-F 0 "#PWR04" H 2850 5300 50  0001 C CNN
-F 1 "GND" H 2850 5400 50  0000 C CNN
-F 2 "" H 2850 5550 60  0000 C CNN
-F 3 "" H 2850 5550 60  0000 C CNN
-	1    2850 5550
+P 2850 5600
+F 0 "#PWR04" H 2850 5350 50  0001 C CNN
+F 1 "GND" H 2850 5450 50  0000 C CNN
+F 2 "" H 2850 5600 60  0000 C CNN
+F 3 "" H 2850 5600 60  0000 C CNN
+	1    2850 5600
 	1    0    0    -1
 $EndComp
@@
 NoConn ~ 2550 3900
 Wire Wire Line
-	4750 4300 4750 4350
-Wire Wire Line
-	3200 6000 3200 5550
-Wire Wire Line
-	2900 6000 2900 5800
+	4750 4250 4750 4350
+Wire Wire Line
+	3200 5550 3200 6100
+Wire Wire Line
+	2900 5800 2900 6100
 Wire Wire Line
 	2900 5800 3050 5800
@@
 	3350 5800 3500 5800
 Wire Wire Line
-	3500 5800 3500 6000
-Wire Wire Line
-	3500 6700 3500 6500
-Wire Wire Line
-	3200 6500 3200 6700
-Wire Wire Line
-	2900 6700 2900 6500
+	3500 5800 3500 6100
+Wire Wire Line
+	3500 6400 3500 6700
+Wire Wire Line
+	3200 6400 3200 6700
+Wire Wire Line
+	2900 6400 2900 6700
 Wire Wire Line
 	3650 7250 3650 7300
@@
 	3750 5800 3650 5800
 Wire Wire Line
+	3800 5800 3950 5800
+Wire Wire Line
+	3950 5800 3950 6050
+Wire Wire Line
+	2550 3750 2500 3750
+Wire Wire Line
+	4750 3950 4750 3800
+Connection ~ 4750 3900
+$Comp
+L RN4020 U1
+U 1 1 561FC38B
+P 3450 4400
+F 0 "U1" H 2800 5350 60  0001 C CNN
+F 1 "RN4020" H 3950 5350 60  0000 C CNN
+F 2 "" H 3950 5350 60  0001 C CNN
+F 3 "" H 3950 5350 60  0000 C CNN
+	1    3450 4400
+	1    0    0    -1
+$EndComp
+Wire Wire Line
+	2850 5550 2850 5600
+Wire Wire Line
+	2350 4350 2550 4350
+Wire Wire Line
+	2350 4500 2550 4500
+Wire Wire Line
+	2350 4650 2550 4650
+Wire Wire Line
+	2350 4800 2550 4800
+Wire Wire Line
 	3650 5800 3650 5550
 Wire Wire Line
 	3800 5550 3800 5800
 Wire Wire Line
-	3800 5800 3950 5800
-Wire Wire Line
-	3950 5800 3950 6050
-Wire Wire Line
-	2550 4350 2350 4350
-Wire Wire Line
-	2350 4500 2550 4500
-Wire Wire Line
-	2550 4650 2350 4650
-Wire Wire Line
-	2350 4800 2550 4800
-Wire Wire Line
-	4750 3800 4750 3900
+	4000 5600 4000 5550
 Wire Wire Line
 	4750 3900 4300 3900
-Wire Wire Line
-	2550 3750 2500 3750
 $EndSCHEMATC

Commit message: Footprints
Parts:
- C1: footprint Capacitors_Tantalum_SMD:TantalC_SizeA_EIA-3216_HandSoldering -> (none)
- R1, R2, R3: footprint Resistors_SMD:R_1206_HandSoldering -> (none)
Changed lines of the file:
@@
 F 0 "R1" V 2980 6250 40  0000 C CNN
 F 1 "R" V 2907 6251 40  0000 C CNN
-F 2 "Resistors_SMD:R_1206_HandSoldering" V 2800 6250 30  0000 C CNN
+F 2 "" V 2800 6250 30  0000 C CNN
 F 3 "~" H 2900 6250 30  0000 C CNN
 	1    2900 6250
@@
 F 0 "C1" H 4750 4200 40  0001 L CNN
 F 1 "C" H 4756 4015 40  0000 L CNN
-F 2 "Capacitors_Tantalum_SMD:TantalC_SizeA_EIA-3216_HandSoldering" H 4788 3950 30  0000 C CNN
+F 2 "" H 4788 3950 30  0000 C CNN
 F 3 "~" H 4750 4100 60  0000 C CNN
 	1    4750 4100
@@
 F 0 "D1" H 2900 7000 50  0000 C CNN
 F 1 "LED" H 2900 6800 50  0000 C CNN
-F 2 "" H 2900 6900 60  0000 C CNN
+F 2 "" H 2900 6900 60  0001 C CNN
 F 3 "~" H 2900 6900 60  0000 C CNN
 	1    2900 6900
@@
 F 0 "R2" V 3280 6250 40  0000 C CNN
 F 1 "R" V 3207 6251 40  0000 C CNN
-F 2 "Resistors_SMD:R_1206_HandSoldering" V 3130 6250 30  0000 C CNN
+F 2 "" V 3130 6250 30  0000 C CNN
 F 3 "~" H 3200 6250 30  0000 C CNN
 	1    3200 6250
@@
 F 0 "R3" V 3580 6250 40  0000 C CNN
 F 1 "R" V 3507 6251 40  0000 C CNN
-F 2 "Resistors_SMD:R_1206_HandSoldering" V 3430 6250 30  0000 C CNN
+F 2 "" V 3430 6250 30  0000 C CNN
 F 3 "~" H 3500 6250 30  0000 C CNN
 	1    3500 6250
@@
 F 0 "D2" H 3200 7000 50  0000 C CNN
 F 1 "LED" H 3200 6800 50  0000 C CNN
-F 2 "" H 3200 6900 60  0000 C CNN
+F 2 "" H 3200 6900 60  0001 C CNN
 F 3 "~" H 3200 6900 60  0000 C CNN
 	1    3200 6900
@@
 F 0 "D3" H 3500 7000 50  0000 C CNN
 F 1 "LED" H 3500 6800 50  0000 C CNN
-F 2 "" H 3500 6900 60  0000 C CNN
+F 2 "" H 3500 6900 60  0001 C CNN
 F 3 "~" H 3500 6900 60  0000 C CNN
 	1    3500 6900

Commit message: Footprint RN4020
Parts:
- removed C1: C, symbol C
- added C1: CP1, Capacitors_Tantalum_SMD:TantalC_SizeB_EIA-3528_HandSoldering, symbol CP1
- D1, D2, D3: footprint (none) -> LEDs:LED-3MM
- R1, R2, R3: footprint (none) -> Resistors_SMD:R_1206_HandSoldering
- U1: footprint (none) -> RN4020:RN4020
Connections:
- net +3V3: now also C1.1
- net GND: now also C1.2
Changed lines of the file:
@@
 F 0 "R1" V 2980 6250 40  0000 C CNN
 F 1 "R" V 2907 6251 40  0000 C CNN
-F 2 "" V 2800 6250 30  0000 C CNN
+F 2 "Resistors_SMD:R_1206_HandSoldering" V 2800 6250 30  0001 C CNN
 F 3 "~" H 2900 6250 30  0000 C CNN
 	1    2900 6250
-	1    0    0    -1
-$EndComp
-$Comp
-L C C1
-U 1 1 561FB9E8
-P 4750 4100
-F 0 "C1" H 4750 4200 40  0001 L CNN
-F 1 "C" H 4756 4015 40  0000 L CNN
-F 2 "" H 4788 3950 30  0000 C CNN
-F 3 "~" H 4750 4100 60  0000 C CNN
-	1    4750 4100
 	1    0    0    -1
 $EndComp
@@
 F 0 "D1" H 2900 7000 50  0000 C CNN
 F 1 "LED" H 2900 6800 50  0000 C CNN
-F 2 "" H 2900 6900 60  0001 C CNN
+F 2 "LEDs:LED-3MM" H 2900 6900 60  0001 C CNN
 F 3 "~" H 2900 6900 60  0000 C CNN
 	1    2900 6900
@@
 F 0 "R2" V 3280 6250 40  0000 C CNN
 F 1 "R" V 3207 6251 40  0000 C CNN
-F 2 "" V 3130 6250 30  0000 C CNN
+F 2 "Resistors_SMD:R_1206_HandSoldering" V 3130 6250 30  0001 C CNN
 F 3 "~" H 3200 6250 30  0000 C CNN
 	1    3200 6250
@@
 F 0 "R3" V 3580 6250 40  0000 C CNN
 F 1 "R" V 3507 6251 40  0000 C CNN
-F 2 "" V 3430 6250 30  0000 C CNN
+F 2 "Resistors_SMD:R_1206_HandSoldering" V 3430 6250 30  0001 C CNN
 F 3 "~" H 3500 6250 30  0000 C CNN
 	1    3500 6250
@@
 F 0 "D2" H 3200 7000 50  0000 C CNN
 F 1 "LED" H 3200 6800 50  0000 C CNN
-F 2 "" H 3200 6900 60  0001 C CNN
+F 2 "LEDs:LED-3MM" H 3200 6900 60  0001 C CNN
 F 3 "~" H 3200 6900 60  0000 C CNN
 	1    3200 6900
@@
 F 0 "D3" H 3500 7000 50  0000 C CNN
 F 1 "LED" H 3500 6800 50  0000 C CNN
-F 2 "" H 3500 6900 60  0001 C CNN
+F 2 "LEDs:LED-3MM" H 3500 6900 60  0001 C CNN
 F 3 "~" H 3500 6900 60  0000 C CNN
 	1    3500 6900
@@
 F 0 "U1" H 2800 5350 60  0001 C CNN
 F 1 "RN4020" H 3950 5350 60  0000 C CNN
-F 2 "" H 3950 5350 60  0001 C CNN
+F 2 "RN4020:RN4020" H 3950 5350 60  0001 C CNN
 F 3 "" H 3950 5350 60  0000 C CNN
 	1    3450 4400
@@
 Wire Wire Line
 	4750 3900 4300 3900
+$Comp
+L CP1 C1
+U 1 1 5637C0B9
+P 4750 4100
+F 0 "C1" H 4775 4200 50  0000 L CNN
+F 1 "CP1" H 4775 4000 50  0000 L CNN
+F 2 "Capacitors_Tantalum_SMD:TantalC_SizeB_EIA-3528_HandSoldering" H 4750 4100 60  0001 C CNN
+F 3 "" H 4750 4100 60  0000 C CNN
+	1    4750 4100
+	1    0    0    -1
+$EndComp
 $EndSCHEMATC

Commit message: 50% Poncho
Parts:
- C1: footprint Capacitors_Tantalum_SMD:TantalC_SizeB_EIA-3528_HandSoldering -> Capacitors_Tantalum_SMD:TantalC_SizeB_EIA-3528_Reflow
- R1, R2, R3: footprint Resistors_SMD:R_1206_HandSoldering -> Resistors_SMD:R_1206
Changed lines of the file:
@@
 F 0 "R1" V 2980 6250 40  0000 C CNN
 F 1 "R" V 2907 6251 40  0000 C CNN
-F 2 "Resistors_SMD:R_1206_HandSoldering" V 2800 6250 30  0001 C CNN
+F 2 "Resistors_SMD:R_1206" V 2800 6250 30  0001 C CNN
 F 3 "~" H 2900 6250 30  0000 C CNN
 	1    2900 6250
@@
 F 0 "R2" V 3280 6250 40  0000 C CNN
 F 1 "R" V 3207 6251 40  0000 C CNN
-F 2 "Resistors_SMD:R_1206_HandSoldering" V 3130 6250 30  0001 C CNN
+F 2 "Resistors_SMD:R_1206" V 3130 6250 30  0001 C CNN
 F 3 "~" H 3200 6250 30  0000 C CNN
 	1    3200 6250
@@
 F 0 "R3" V 3580 6250 40  0000 C CNN
 F 1 "R" V 3507 6251 40  0000 C CNN
-F 2 "Resistors_SMD:R_1206_HandSoldering" V 3430 6250 30  0001 C CNN
+F 2 "Resistors_SMD:R_1206" V 3430 6250 30  0001 C CNN
 F 3 "~" H 3500 6250 30  0000 C CNN
 	1    3500 6250
@@
 F 0 "C1" H 4775 4200 50  0000 L CNN
 F 1 "CP1" H 4775 4000 50  0000 L CNN
-F 2 "Capacitors_Tantalum_SMD:TantalC_SizeB_EIA-3528_HandSoldering" H 4750 4100 60  0001 C CNN
+F 2 "Capacitors_Tantalum_SMD:TantalC_SizeB_EIA-3528_Reflow" H 4750 4100 60  0001 C CNN
 F 3 "" H 4750 4100 60  0000 C CNN
 	1    4750 4100

Commit message: New Poncho
Parts:
- added XA1: Conn_PonchoMP_2x_20x2, symbol Conn_PonchoMP_2x_20x2
Connections:
- net CMD: now also XA1.74 (GPIO3)
- net CTS: now also XA1.76 (GPIO5)
- net HW: now also XA1.78 (GPIO7)
- net RTS: now also XA1.80 (GPIO8)
- net SW: now also XA1.72 (GPIO1)
- net UART_RX renamed RX
- net RX: now also XA1.23 (RXD)
- net UART_TX renamed TX
- net TX: now also XA1.25 (TXD)
- no-connect marks 6 -> 10
Other:
- moved on the sheet: C1, D1, D2, D3, R1, R2, R3

Commit message: PCB Completa
Parts:
- added unit 2 of XA1
Connections:
- net +3V3: now also XA1.41 (+3.3V)
- net GND: now also XA1.79 (GND)
- no-connect marks 10 -> 21
Changed lines of the file:
@@
 $EndComp
 $Comp
-L +3.3V #PWR01
+L +3.3V #PWR6
 U 1 1 561FB9EF
 P 7250 2100
-F 0 "#PWR01" H 7250 2060 30  0001 C CNN
+F 0 "#PWR6" H 7250 2060 30  0001 C CNN
 F 1 "+3.3V" H 7250 2210 30  0000 C CNN
 F 2 "" H 7250 2100 60  0000 C CNN
@@
 $EndComp
 $Comp
-L GND #PWR02
+L GND #PWR7
 U 1 1 561FCE9A
 P 7250 2650
-F 0 "#PWR02" H 7250 2400 50  0001 C CNN
+F 0 "#PWR7" H 7250 2400 50  0001 C CNN
 F 1 "GND" H 7250 2500 50  0000 C CNN
 F 2 "" H 7250 2650 60  0000 C CNN
@@
 $EndComp
 $Comp
-L GND #PWR03
+L GND #PWR4
 U 1 1 561FD06E
 P 6500 3900
-F 0 "#PWR03" H 6500 3650 50  0001 C CNN
+F 0 "#PWR4" H 6500 3650 50  0001 C CNN
 F 1 "GND" H 6500 3750 50  0000 C CNN
 F 2 "" H 6500 3900 60  0000 C CNN
@@
 $EndComp
 $Comp
-L GND #PWR04
+L GND #PWR2
 U 1 1 561FD154
 P 5350 3900
-F 0 "#PWR04" H 5350 3650 50  0001 C CNN
+F 0 "#PWR2" H 5350 3650 50  0001 C CNN
 F 1 "GND" H 5350 3750 50  0000 C CNN
 F 2 "" H 5350 3900 60  0000 C CNN
@@
 $EndComp
 $Comp
-L GND #PWR05
+L GND #PWR1
 U 1 1 561FD233
 P 5000 2050
-F 0 "#PWR05" H 5000 1800 50  0001 C CNN
+F 0 "#PWR1" H 5000 1800 50  0001 C CNN
 F 1 "GND" H 5000 1900 50  0000 C CNN
 F 2 "" H 5000 2050 60  0000 C CNN
@@
 $EndComp
 $Comp
-L GND #PWR06
+L GND #PWR5
 U 1 1 561FD25C
 P 6800 2050
-F 0 "#PWR06" H 6800 1800 50  0001 C CNN
+F 0 "#PWR5" H 6800 1800 50  0001 C CNN
 F 1 "GND" H 6800 1900 50  0000 C CNN
 F 2 "" H 6800 2050 60  0000 C CNN
@@
 $EndComp
 $Comp
-L GND #PWR07
+L GND #PWR3
 U 1 1 561FD579
 P 6150 5600
-F 0 "#PWR07" H 6150 5350 50  0001 C CNN
+F 0 "#PWR3" H 6150 5350 50  0001 C CNN
 F 1 "GND" H 6150 5450 50  0000 C CNN
 F 2 "" H 6150 5600 60  0000 C CNN
@@
 Wire Wire Line
 	8200 3450 8300 3450
+$Comp
+L Conn_PonchoMP_2x_20x2 XA1
+U 2 1 5640D5F7
+P 8400 2150
+F 0 "XA1" H 8400 2700 60  0000 C CNN
+F 1 "Conn_PonchoMP_2x_20x2" H 8400 2600 60  0000 C CNN
+F 2 "" H 8250 2500 60  0000 C CNN
+F 3 "" H 8250 2500 60  0000 C CNN
+	2    8400 2150
+	1    0    0    -1
+$EndComp
+NoConn ~ 7950 1950
+NoConn ~ 7950 2050
+NoConn ~ 7950 2150
+NoConn ~ 7950 2250
+NoConn ~ 7950 2350
+NoConn ~ 8850 2450
+NoConn ~ 8850 2350
+NoConn ~ 8850 2250
+NoConn ~ 8850 2150
+NoConn ~ 8850 2050
+NoConn ~ 8850 1950
+$Comp
+L +3.3V #PWR8
+U 1 1 5640DA42
+P 7950 1850
+F 0 "#PWR8" H 7950 1700 50  0001 C CNN
+F 1 "+3.3V" H 7950 1990 50  0000 C CNN
+F 2 "" H 7950 1850 60  0000 C CNN
+F 3 "" H 7950 1850 60  0000 C CNN
+	1    7950 1850
+	0    -1   -1   0
+$EndComp
+$Comp
+L GND #PWR9
+U 1 1 5640DA6A
+P 8850 1850
+F 0 "#PWR9" H 8850 1600 50  0001 C CNN
+F 1 "GND" H 8850 1700 50  0000 C CNN
+F 2 "" H 8850 1850 60  0000 C CNN
+F 3 "" H 8850 1850 60  0000 C CNN
+	1    8850 1850
+	0    -1   -1   0
+$EndComp
 $EndSCHEMATC

Commit message: Footprint acondicionandose
Connections:
- net RX: now also U1.5 (UART_TX); no longer U1.6 (UART_RX)
- net TX: now also U1.6 (UART_RX); no longer U1.5 (UART_TX)
Changed lines of the file:
@@
 Text GLabel 3950 2600 2    60   Input ~ 0
 RX
+Text GLabel 5000 2800 0    60   Input ~ 0
+TX
 Text GLabel 5000 2650 0    60   Input ~ 0
-TX
-Text GLabel 5000 2800 0    60   Input ~ 0
 RX
 Wire Wire Line
